File: daughter/rev1/monitor.kicad_sch (KiCad schematic)
At the start: 18 parts, among them U13 ADS8568SPM

Commit message: Change adc driver to ADA4945
Parts:
- U13: footprint ADS8568SPM:QFP50P1200X1200X160-64N -> myparts:QFP50P1200X1200X160-64N
Changed lines of the file:
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@@
 		)
 		(instances
-			(project ""
+			(project "psc_daughter_brd"
 				(path "/40891cc8-bf64-41f4-8f69-a607d7b280eb/79a78ff4-0a06-4569-970f-a218b7d7f7b9"
 					(reference "#PWR0142")
@@
 			)
 		)
-		(property "Footprint" "ADS8568SPM:QFP50P1200X1200X160-64N"
+		(property "Footprint" "myparts:QFP50P1200X1200X160-64N"
 			(at 254 135.89 0)
 			(effects
@@
 		)
 		(instances
-			(project ""
+			(project "psc_daughter_brd"
 				(path "/40891cc8-bf64-41f4-8f69-a607d7b280eb/79a78ff4-0a06-4569-970f-a218b7d7f7b9"
 					(reference "U13")
@@
 		)
 		(instances
-			(project ""
+			(project "psc_daughter_brd"
 				(path "/40891cc8-bf64-41f4-8f69-a607d7b280eb/79a78ff4-0a06-4569-970f-a218b7d7f7b9"
 					(reference "#PWR097")
@@
 		)
 		(instances
-			(project ""
+			(project "psc_daughter_brd"
 				(path "/40891cc8-bf64-41f4-8f69-a607d7b280eb/79a78ff4-0a06-4569-970f-a218b7d7f7b9"
 					(reference "#PWR0262")
@@
 		)
 		(instances
-			(project ""
+			(project "psc_daughter_brd"
 				(path "/40891cc8-bf64-41f4-8f69-a607d7b280eb/79a78ff4-0a06-4569-970f-a218b7d7f7b9"
 					(reference "#PWR0143")
