File: daughter/rev1/psc_daughter_brd.kicad_sch (KiCad schematic)
At the start: 8 parts

Commit message: linked ADR1001 to DCCT ADC reference for 5V and 2.5V
Other:
- sheet DAC ports: added adc_ref_out; removed none
- sheet DCCT ADCs ports: added adc_ref_in; removed none
Changed lines of the file:
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@@
+	(wire
+		(pts
+			(xy 149.86 189.23) (xy 161.29 189.23)
+		)
+		(stroke
+			(width 0)
+			(type default)
+		)
+	)
 	(wire
 		(pts
@@
 	(wire
 		(pts
+			(xy 161.29 111.76) (xy 149.86 111.76)
+		)
+		(stroke
+			(width 0)
+			(type default)
+		)
+	)
+	(wire
+		(pts
 			(xy 128.27 73.66) (xy 162.56 73.66)
 		)
@@
 		(pts
 			(xy 334.01 179.07) (xy 334.01 177.8)
+		)
+		(stroke
+			(width 0)
+			(type default)
+		)
+	)
+	(wire
+		(pts
+			(xy 149.86 111.76) (xy 149.86 189.23)
 		)
 		(stroke
@@
 			)
 		)
+		(pin "adc_ref_in" input
+			(at 161.29 189.23 180)
+			(effects
+				(font
+					(size 1.27 1.27)
+				)
+				(justify left)
+			)
+		)
 		(instances
 			(project "psc_daughter_brd"
@@
 			(effects
 				(font
+					(size 1.27 1.27)
+				)
+				(justify left)
+			)
+		)
+		(pin "adc_ref_out" input
+			(at 161.29 111.76 180)
+			(effects
+				(font
