File: daughter/rev1/dac.kicad_sch (KiCad schematic)
At the start: 46 parts, among them U10 BUF634AIDR, U11 BUF634AIDR, U3 AD8676ARZ, U5 AD5791BRUZ, U6 AD797ARZ, U7 OPA277, U9 OPA277

Commit message: linked ADR1001 to DCCT ADC reference for 5V and 2.5V
Other:
- sheet Voltage Reference ports: added adc_ref_out; removed none
Changed lines of the file:
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@@
 	(wire
 		(pts
+			(xy 40.64 39.37) (xy 48.26 39.37)
+		)
+		(stroke
+			(width 0)
+			(type default)
+		)
+	)
+	(wire
+		(pts
 			(xy 102.87 138.43) (xy 106.68 138.43)
 		)
@@
 		)
 	)
+	(hierarchical_label "adc_ref_out"
+		(shape input)
+		(at 48.26 39.37 0)
+		(effects
+			(font
+				(size 1.27 1.27)
+			)
+			(justify left)
+		)
+	)
 	(hierarchical_label "dac_out+"
 		(shape input)
@@
 			(effects
 				(font
+					(size 1.27 1.27)
+				)
+				(justify right)
+			)
+		)
+		(pin "adc_ref_out" input
+			(at 40.64 39.37 0)
+			(effects
+				(font

Commit message: DAC fix pin 10 IOvcc was tied to 1.8V should be tied to 3.3V
Connections:
- net +1.8V is gone; now on net +3.3V: C29.1, U5.10 (IOV_{CC})
Changed lines of the file:
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@@
 	)
 	(junction
+		(at 66.04 72.39)
+		(diameter 0)
+		(color 0 0 0 0)
+	)
+	(junction
 		(at 264.16 115.57)
 		(diameter 0)
@@
 	(wire
 		(pts
+			(xy 66.04 72.39) (xy 66.04 88.9)
+		)
+		(stroke
+			(width 0)
+			(type default)
+		)
+	)
+	(wire
+		(pts
 			(xy 40.64 39.37) (xy 48.26 39.37)
 		)
@@
 	(wire
 		(pts
-			(xy 66.04 59.69) (xy 66.04 88.9)
-		)
-		(stroke
-			(width 0)
-			(type default)
-		)
-	)
-	(wire
-		(pts
 			(xy 257.81 182.88) (xy 262.89 182.88)
 		)
@@
 	(wire
 		(pts
+			(xy 66.04 59.69) (xy 66.04 72.39)
+		)
+		(stroke
+			(width 0)
+			(type default)
+		)
+	)
+	(wire
+		(pts
 			(xy 298.45 182.88) (xy 298.45 199.39)
 		)
@@
 	(wire
 		(pts
-			(xy 80.01 69.85) (xy 80.01 72.39)
-		)
-		(stroke
-			(width 0)
-			(type default)
-		)
-	)
-	(wire
-		(pts
 			(xy 298.45 182.88) (xy 298.45 179.07)
 		)
@@
 	(wire
 		(pts
+			(xy 66.04 72.39) (xy 80.01 72.39)
+		)
+		(stroke
+			(width 0)
+			(type default)
+		)
+	)
+	(wire
+		(pts
 			(xy 196.85 115.57) (xy 200.66 115.57)
 		)
@@
 					(unit 1)
 				)
-			)
-		)
-	)
-	(symbol
-		(lib_id "PSC:+1.8V")
-		(at 80.01 69.85 0)
-		(unit 1)
-		(exclude_from_sim no)
-		(in_bom yes)
-		(on_board yes)
-		(dnp no)
-		(fields_autoplaced yes)
-		(property "Reference" "#PWR054"
-			(at 80.01 73.66 0)
-			(effects
-				(font
-					(size 1.27 1.27)
-				)
-				(hide yes)
-			)
-		)
-		(property "Value" "+1.8V"
-			(at 80.01 64.77 0)
-			(effects
-				(font
-					(size 1.27 1.27)
-				)
-			)
-		)
-		(property "Footprint" ""
-			(at 80.01 69.85 0)
-			(effects
-				(font
-					(size 1.27 1.27)
-				)
-				(hide yes)
-			)
-		)
-		(property "Datasheet" ""
-			(at 80.01 69.85 0)
-			(effects
-				(font
-					(size 1.27 1.27)
-				)
-				(hide yes)
-			)
-		)
-		(property "Description" ""
-			(at 80.01 69.85 0)
-			(effects
-				(font
-					(size 1.27 1.27)
-				)
-				(hide yes)
-			)
-		)
-		(pin "1"
-		)
-		(instances
-			(project "psc_daughter_brd"
-				(path "/40891cc8-bf64-41f4-8f69-a607d7b280eb/dea95122-986e-41c8-b99e-e429cc6f4cd5"
-					(reference "#PWR054")
-					(unit 1)
-				)
