File: daughter/rev1/digout.kicad_sch (KiCad schematic)
At the start: 17 parts, among them U38 TXUN0104RUTR, U39 ADUM5240ARZ, U40 ADUM5240ARZ

Commit message: Change adc driver to ADA4945
Parts:
- U39, U40: footprint myparts:R_8_ADI-M -> myparts:R_8_ADI
Changed lines of the file:
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@@
 			)
 		)
-		(property "Footprint" "myparts:R_8_ADI-M"
+		(property "Footprint" "myparts:R_8_ADI"
 			(at 127 50.8 0)
 			(effects
@@
 		)
 		(instances
-			(project ""
+			(project "psc_daughter_brd"
 				(path "/40891cc8-bf64-41f4-8f69-a607d7b280eb/979dab62-5512-4152-97ee-117138a961d3/84c3e299-56b9-4043-9091-ed3bb176fd4f"
 					(reference "#PWR0184")
@@
 			)
 		)
-		(property "Footprint" "myparts:R_8_ADI-M"
+		(property "Footprint" "myparts:R_8_ADI"
 			(at 127 120.65 0)
 			(effects
