File: daughter/rev1/psc_daughter_brd.kicad_pcb (KiCad board)
At the start: 10 copper layers, 40 x 160 mm, 326 parts, among them J1 61082-061400LF, J2 61082-061400LF, U1 AD8221, U10 BUF634AIDR, U11 BUF634AIDR, U12 ADR1001AEZ, U13 ADS8568SPM, U14 AD8221, U15 OPA277, U16 AD8221, U17 OPA277, U18 AD8221, U19 OPA277, U2 OPA277, U20 LT3042xMSE, U21 THP210DR, U24 ADA4523-1BRMZ, U25 LT6202CS5, U26 THP210DR, U27 AD8429BRZ, U3 AD8676ARZ, U31 LTC2376CDE-20, U32 LTC6655BHLS8-5, U33 AD8429BRZ, U35 LT6202CS5, U37 LTC2376CDE-20, U38 TXUN0104RUTR, U39 ADUM5240ARZ, U4 AD8676xR, U40 ADUM5240ARZ, U41 TXUN0104RUTR, U42 ADUM5242ARZ, U43 ADUM5242ARZ, U5 AD5791BRUZ, U6 AD797ARZ, U7 OPA277, U8 AD8676xR, U9 OPA277

Commit message: Rename versions
Parts:
- removed C109, C110: 3nF, Capacitor_SMD:C_0603_1608Metric
- removed C111, C112: 2nF, Capacitor_SMD:C_0603_1608Metric
- removed C113, C115, C131, C135, C149, C150: 0.1uF, Capacitor_SMD:C_0402_1005Metric
- removed C114, C118: 10uF, Capacitor_SMD:C_0603_1608Metric
- removed C120, C122, C129: 470pF, Capacitor_SMD:C_0402_1005Metric
- removed C125: 4.7uF, Capacitor_SMD:C_0402_1005Metric
- removed D8, D9: BAT54S, Package_TO_SOT_SMD:SOT-23
- removed R35, R37, R38, R39, R40, R41, R44, R45, R47, R48, R77: 10.0K, Resistor_SMD:R_0603_1608Metric
- removed R49: 1K, Resistor_SMD:R_0402_1005Metric
- removed R74: 750, Resistor_SMD:R_0402_1005Metric
- removed R75: 5.62k, Resistor_SMD:R_0402_1005Metric
- removed R76: 0, Resistor_SMD:R_0402_1005Metric
- removed U21, U26: THP210DR, myparts:SOIC_210DR_TEX
- removed U24: ADA4523-1BRMZ, myparts:RM-8_ADI
- removed U25: LT6202CS5, myparts:LT6202CS5
- removed U4, U8: AD8676xR, Package_SO:SOIC-8_3.9x4.9mm_P1.27mm
- added C161: 10uF, Capacitor_SMD:C_0603_1608Metric, B.Cu at (145.8, 66.0)
- added C163: 0.1uF, Capacitor_SMD:C_0402_1005Metric, B.Cu at (145.8, 69.4)
- added C167: 6800pF, Capacitor_SMD:C_0402_1005Metric, F.Cu at (150.5, 81.2)
- added C168: 3300pF, Capacitor_SMD:C_0402_1005Metric, F.Cu at (148.5, 81.2)
- added C169: 6800pF, Capacitor_SMD:C_0402_1005Metric, F.Cu at (146.6, 81.2)
- added C175: 6800pF, Capacitor_SMD:C_0402_1005Metric, F.Cu at (150.6, 89.3)
- added U28: AD8675ARZ, Package_SO:SOIC-8_3.9x4.9mm_P1.27mm, F.Cu at (157.6, 75.5)
- added U30: LTC6363IMS8, Package_SO:MSOP-8_3x3mm_P0.65mm, F.Cu at (157.5, 84.3)
- added U34: AD8675ARZ, Package_SO:SOIC-8_3.9x4.9mm_P1.27mm, F.Cu at (148.7, 75.3)
- added U36: LTC6363IMS8, Package_SO:MSOP-8_3x3mm_P0.65mm, F.Cu at (148.5, 84.1)
- C124: value 0.1uF -> 0.01uF
- C128: value 470pF -> 0.1uF; moved to B.Cu
- C132: value 47nF -> 6800pF
- C133: value 47uF -> 3300pF; footprint Capacitor_SMD:C_1210_3225Metric -> Capacitor_SMD:C_0402_1005Metric; moved to F.Cu
- C134: value 10uF -> 6800pF; footprint Capacitor_SMD:C_0603_1608Metric -> Capacitor_SMD:C_0402_1005Metric
- C137: value 0.1uF -> 10uF; footprint Capacitor_SMD:C_0402_1005Metric -> Capacitor_SMD:C_0603_1608Metric
- C138: value 6800pF -> 0.1uF; moved to B.Cu
- C139: value 10uF -> 0.1uF; footprint Capacitor_SMD:C_0603_1608Metric -> Capacitor_SMD:C_0402_1005Metric
- C155, C157: moved to F.Cu
- C159: value 0.1uF -> 0.01uF; moved to F.Cu
- R46, R58: value 10.0K -> 1.3K; footprint Resistor_SMD:R_0603_1608Metric -> Resistor_SMD:R_0402_1005Metric
- R50: value 2 -> 10
- R51, R63: value 10.0K -> 15; footprint Resistor_SMD:R_0603_1608Metric -> Resistor_SMD:R_0402_1005Metric
- R59, R60: value 10.0K -> 10K; footprint Resistor_SMD:R_0603_1608Metric -> Resistor_SMD:R_0402_1005Metric
- R62: value 10.0K -> 10; footprint Resistor_SMD:R_0603_1608Metric -> Resistor_SMD:R_0402_1005Metric
- moved C124 43.5 mm to (156.6, 70.8)
- moved C126 41.2 mm to (154.2, 72.0), turned to 90 degrees
- moved R50 21.4 mm to (158.5, 80.3), turned to 180 degrees
- moved C132 20.3 mm to (159.5, 81.4), turned to 180 degrees
- moved C134 19.4 mm to (155.5, 81.4), turned to 180 degrees
- moved C173 16.8 mm to (146.1, 84.9), turned to -90 degrees
- moved C171 13.8 mm to (147.6, 85.3)
- moved C133 13.7 mm to (157.5, 81.4), turned to 180 degrees
- moved C127 13.6 mm to (160.1, 75.9), turned to 0 degrees
- moved C137 13.5 mm to (158.3, 85.5)
- moved C136 13.1 mm to (156.6, 85.4)
- moved C159 13.0 mm to (147.7, 70.6), turned to 180 degrees
- moved R58 12.1 mm to (149.9, 70.6), turned to 0 degrees
- moved C130 11.9 mm to (156.7, 75.9), turned to 180 degrees
- moved C157 11.4 mm to (145.1, 91.9), turned to 90 degrees
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Connections:
- net /DAC/adc_ref_out renamed /DCCT ADCs/DCCT Channel 1/adc_vref
- C124 pad 1: Net-(U24-*SD) -> Net-(U28-+)
- C124 pad 2: Net-(U24-SDC) -> GND
- C126 pad 1: +15V -> -15V
- C127 pad 1: +5.3VA -> +15V
- C128 pad 1: Net-(U26-IN+) -> -15V
- C128 pad 2: Net-(U26-OUT-) -> GND
- C130 pad 1: +5.3VA -> +15V
- C132 pad 1: Net-(C132-Pad1) -> GND
- C133 pad 1: GND -> Net-(C132-Pad2)
- C134 pad 1: +15V -> Net-(C133-Pad2)
- C137 pad 1: +5.3VA -> -5.3VA
- C138 pad 1: GND -> +5.3VA
- C138 pad 2: Net-(U37-IN+) -> GND
- C159 pad 1: /DCCT ADCs/DCCT Channel 1/drv_vref -> Net-(U34-+)
- C162 pad 1: +5.3VA -> +15V
- C165 pad 1: +5.3VA -> +15V
- C189 pad 1: +1.8V -> +1V8
- C29 pad 1: +3.3V -> +1.8V
- R46 pad 1: Net-(U26-IN+) -> Net-(U28-+)
- R46 pad 2: Net-(C112-Pad2) -> Net-(R46-Pad2)
- R50 pad 1: Net-(C133-Pad2) -> Net-(C132-Pad2)
- R50 pad 2: Net-(C132-Pad2) -> Net-(U28--)
- R51 pad 1: Net-(U21-IN-) -> Net-(C133-Pad2)
- R52 pad 2: Net-(U26-OUT-) -> Net-(R52-Pad2)
- R53 pad 2: Net-(U26-OUT+) -> Net-(R53-Pad2)
- R58 pad 1: Net-(U26-IN-) -> Net-(U34-+)
- R58 pad 2: GND -> Net-(R58-Pad2)
- R60 pad 1: GND -> Net-(U35-+)
- R60 pad 2: Net-(U35-+) -> GND
- R62 pad 1: Net-(U21-OUT+) -> Net-(C167-Pad2)
- R62 pad 2: Net-(U21-IN-) -> Net-(U34--)
- R63 pad 1: Net-(U26-OUT+) -> Net-(C168-Pad2)
- R63 pad 2: Net-(U26-IN-) -> GND
- R65 pad 2: Net-(U21-OUT+) -> Net-(R65-Pad2)
- U27 pad 7: Net-(D9-COM) -> Net-(R46-Pad2)
- U33 pad 7: Net-(D8-COM) -> Net-(R58-Pad2)
- U41 pad 11: +1.8V -> +1V8
- U5 pad 10: +3.3V -> +1.8V
Routing:
- net Net-(C110-Pad2): track 17.8 -> 0.00 mm, vias 2 -> 0
- net Net-(C109-Pad2): track 17.8 -> 0.00 mm, vias 2 -> 0
- net GND: track 444.1 -> 426.4 mm, vias 286 -> 290
- net Net-(C111-Pad2): track 16.7 -> 0.00 mm, vias 2 -> 0
- net Net-(C112-Pad2): track 16.7 -> 0.00 mm, vias 2 -> 0
- net Net-(U12-BUF_INP): track 20.9 -> 4.39 mm, vias 2 -> 1
- net Net-(U21-OUT+): track 15.6 -> 0.00 mm
- net Net-(U26-OUT-): track 14.9 -> 0.00 mm
- net Net-(U26-OUT+): track 14.7 -> 0.00 mm
- net Net-(C133-Pad2): track 17.9 -> 4.30 mm, vias 1 -> 0
- net +5.3VA: track 27.2 -> 14.0 mm, vias 11 -> 5
- net -5.3VA: track 24.5 -> 11.5 mm, vias 8 -> 4
- net Net-(R64-Pad2): track 14.7 -> 3.42 mm
- net Net-(U25-+): track 10.7 -> 0.00 mm, vias 2 -> 0
- net Net-(U8B--): track 9.97 -> 0.00 mm
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- added copper zone on In2.Cu, net -5.3VA
- added copper zone on In7.Cu, net /DCCT ADCs/dcct_busy
- removed copper zone on In7.Cu, net -5.3VA
Other:
- board text added: "NSLS-II zuPSC Regulator Board Rev 1 1-5-26"
- board text removed: "NSLS-II zuPSC Regulator Board Rev 2 8-17-26"
