File: carrier/revA/psc_carrier_brd.kicad_pcb (KiCad board)
At the start: 10 copper layers, 241.3 x 255 mm, 243 parts, among them J1 6469028-1, J10 61083-061402LF, J11 0836149012, J12 61083-061402LF, J13 61083-061402LF, J14 0836149012, J15 61083-061402LF, J16 61083-061402LF, J17 0836149012, J2 6469028-1, J3 6469028-1, J4 39301022, J5 61083-061402LF, J6 61083-061402LF, J7 1731130154, J8 0836149012, J9 61083-061402LF, Q1 NX7002BKW, U1 3-641215-6, U10 LT3045xDD, U11 LT8643S, U12 LTC2991CMS_TRPBF, U13 LTC2991CMS_TRPBF, U14 LTC2991CMS_TRPBF, U15 Burden, U16 Burden, U17 Burden, U18 Burden, U19 LT1963AEQ, U2 LT1963AEQ, U20 LT3015EQ-15, U21 LT6106, U22 LT6106, U23 CD74HC4050, U3 LT3015EQ-15, U4 LT6106, U5 LT6106, U6 LT3015EDDPBF, U7 LT3045xDD, U8 LT3045xDD, U9 LT3045xDD

Commit message: Add Edmundo PS connectors
Parts:
- removed REF** (x2): AMPHENOL_ICD26S13E6GV00LF, myparts:AMPHENOL_ICD26S13E6GV00LF
- J11, J14, J17, J8: value 0836149012 -> ICD26S13E6GV00LF; footprint myparts:0836149012 -> myparts:AMPHENOL_ICD26S13E6GV00LF
- moved TP15 11.9 mm to (69.3, 108.9)
- moved MT4 10.0 mm to (299.9, 95.0)
- moved MT6 10.0 mm to (68.8, 95.0)
- moved J11 1.50 mm to (140.0, 91.5)
- moved J14 1.50 mm to (185.0, 91.5)
- moved J17 1.50 mm to (230.0, 91.5)
- moved J8 1.50 mm to (95.0, 91.5)
Connections:
- J11 pad 1: /Ch2 Daughterboard/reg.out+ -> /Ch2 Daughterboard/digout.rtn
- J11 pad 10: /Ch2 Daughterboard/digout.spare -> /Ch2 Daughterboard/digin.rtn
- J11 pad 11: /Ch2 Daughterboard/digout.rtn -> /Ch2 Daughterboard/digin.rtn
- J11 pad 12: /Ch2 Daughterboard/digout.rtn -> /Ch2 Daughterboard/digout.spare
- J11 pad 13: unconnected-(J11-Pad13) -> /Ch2 Daughterboard/digout.on2
- J11 pad 14: /Ch2 Daughterboard/reg.out- -> unconnected-(J11-Pad14)
- J11 pad 15: unconnected-(J11-Pad15) -> /Ch2 Daughterboard/ps.ignd-
- J11 pad 16: /Ch2 Daughterboard/ps.vout- -> /Ch2 Daughterboard/ps.spare-
- J11 pad 17: /Ch2 Daughterboard/ps.ignd- -> /Ch2 Daughterboard/ps.vout-
- J11 pad 18: /Ch2 Daughterboard/ps.spare- -> /Ch2 Daughterboard/reg.out-
- J11 pad 19: unconnected-(J11-Pad19) -> /Ch2 Daughterboard/digin.acon
- J11 pad 2: unconnected-(J11-Pad2) -> /Ch2 Daughterboard/digout.rtn
- J11 pad 20: /Ch2 Daughterboard/digin.acon -> /Ch2 Daughterboard/digin.flt1
- J11 pad 21: /Ch2 Daughterboard/digin.flt1 -> /Ch2 Daughterboard/digin.flt2
- J11 pad 22: /Ch2 Daughterboard/digin.flt2 -> /Ch2 Daughterboard/digin.spare
- J11 pad 23: /Ch2 Daughterboard/digin.spare -> unconnected-(J11-Pad23)
- J11 pad 24: /Ch2 Daughterboard/digin.rtn -> unconnected-(J11-Pad24)
- J11 pad 25: /Ch2 Daughterboard/digin.rtn -> unconnected-(J11-Pad25)
- J11 pad 26: (no net) -> unconnected-(J11-Pad26)
- J11 pad 3: /Ch2 Daughterboard/ps.vout+ -> /Ch2 Daughterboard/digout.reset
- J11 pad 4: /Ch2 Daughterboard/ps.ignd+ -> /Ch2 Daughterboard/digout.on1
- J11 pad 5: /Ch2 Daughterboard/ps.spare+ -> unconnected-(J11-Pad5)
- J11 pad 6: unconnected-(J11-Pad6) -> /Ch2 Daughterboard/ps.ignd+
- J11 pad 7: /Ch2 Daughterboard/digout.on1 -> /Ch2 Daughterboard/ps.spare+
- J11 pad 8: /Ch2 Daughterboard/digout.on2 -> /Ch2 Daughterboard/ps.vout+
- J11 pad 9: /Ch2 Daughterboard/digout.reset -> /Ch2 Daughterboard/reg.out+
- J14 pad 1: /Ch3 Daughterboard/reg.out+ -> /Ch3 Daughterboard/digout.rtn
- J14 pad 10: /Ch3 Daughterboard/digout.spare -> /Ch3 Daughterboard/digin.rtn
- J14 pad 11: /Ch3 Daughterboard/digout.rtn -> /Ch3 Daughterboard/digin.rtn
- J14 pad 12: /Ch3 Daughterboard/digout.rtn -> /Ch3 Daughterboard/digout.spare
- J14 pad 13: unconnected-(J14-Pad13) -> /Ch3 Daughterboard/digout.on2
- J14 pad 14: /Ch3 Daughterboard/reg.out- -> unconnected-(J14-Pad14)
- J14 pad 15: unconnected-(J14-Pad15) -> /Ch3 Daughterboard/ps.ignd-
- J14 pad 16: /Ch3 Daughterboard/ps.vout- -> /Ch3 Daughterboard/ps.spare-
- J14 pad 17: /Ch3 Daughterboard/ps.ignd- -> /Ch3 Daughterboard/ps.vout-
- J14 pad 18: /Ch3 Daughterboard/ps.spare- -> /Ch3 Daughterboard/reg.out-
- J14 pad 19: unconnected-(J14-Pad19) -> /Ch3 Daughterboard/digin.acon
- J14 pad 2: unconnected-(J14-Pad2) -> /Ch3 Daughterboard/digout.rtn
- J14 pad 20: /Ch3 Daughterboard/digin.acon -> /Ch3 Daughterboard/digin.flt1
- J14 pad 21: /Ch3 Daughterboard/digin.flt1 -> /Ch3 Daughterboard/digin.flt2
- J14 pad 22: /Ch3 Daughterboard/digin.flt2 -> /Ch3 Daughterboard/digin.spare
- J14 pad 23: /Ch3 Daughterboard/digin.spare -> unconnected-(J14-Pad23)
- J14 pad 24: /Ch3 Daughterboard/digin.rtn -> unconnected-(J14-Pad24)
- J14 pad 25: /Ch3 Daughterboard/digin.rtn -> unconnected-(J14-Pad25)
- J14 pad 26: (no net) -> unconnected-(J14-Pad26)
- J14 pad 3: /Ch3 Daughterboard/ps.vout+ -> /Ch3 Daughterboard/digout.reset
- J14 pad 4: /Ch3 Daughterboard/ps.ignd+ -> /Ch3 Daughterboard/digout.on1
- J14 pad 5: /Ch3 Daughterboard/ps.spare+ -> unconnected-(J14-Pad5)
- J14 pad 6: unconnected-(J14-Pad6) -> /Ch3 Daughterboard/ps.ignd+
- J14 pad 7: /Ch3 Daughterboard/digout.on1 -> /Ch3 Daughterboard/ps.spare+
- J14 pad 8: /Ch3 Daughterboard/digout.on2 -> /Ch3 Daughterboard/ps.vout+
- J14 pad 9: /Ch3 Daughterboard/digout.reset -> /Ch3 Daughterboard/reg.out+
- J17 pad 1: /Ch4 Daughterboard/reg.out+ -> /Ch4 Daughterboard/digout.rtn
- J17 pad 10: /Ch4 Daughterboard/digout.spare -> /Ch4 Daughterboard/digin.rtn
- J17 pad 11: /Ch4 Daughterboard/digout.rtn -> /Ch4 Daughterboard/digin.rtn
- J17 pad 12: /Ch4 Daughterboard/digout.rtn -> /Ch4 Daughterboard/digout.spare
- J17 pad 13: unconnected-(J17-Pad13) -> /Ch4 Daughterboard/digout.on2
- J17 pad 14: /Ch4 Daughterboard/reg.out- -> unconnected-(J17-Pad14)
- J17 pad 15: unconnected-(J17-Pad15) -> /Ch4 Daughterboard/ps.ignd-
- J17 pad 16: /Ch4 Daughterboard/ps.vout- -> /Ch4 Daughterboard/ps.spare-
- J17 pad 17: /Ch4 Daughterboard/ps.ignd- -> /Ch4 Daughterboard/ps.vout-
- J17 pad 18: /Ch4 Daughterboard/ps.spare- -> /Ch4 Daughterboard/reg.out-
- J17 pad 19: unconnected-(J17-Pad19) -> /Ch4 Daughterboard/digin.acon
- J17 pad 2: unconnected-(J17-Pad2) -> /Ch4 Daughterboard/digout.rtn
- J17 pad 20: /Ch4 Daughterboard/digin.acon -> /Ch4 Daughterboard/digin.flt1
- J17 pad 21: /Ch4 Daughterboard/digin.flt1 -> /Ch4 Daughterboard/digin.flt2
- J17 pad 22: /Ch4 Daughterboard/digin.flt2 -> /Ch4 Daughterboard/digin.spare
- J17 pad 23: /Ch4 Daughterboard/digin.spare -> unconnected-(J17-Pad23)
- J17 pad 24: /Ch4 Daughterboard/digin.rtn -> unconnected-(J17-Pad24)
- J17 pad 25: /Ch4 Daughterboard/digin.rtn -> unconnected-(J17-Pad25)
- J17 pad 26: (no net) -> unconnected-(J17-Pad26)
- J17 pad 3: /Ch4 Daughterboard/ps.vout+ -> /Ch4 Daughterboard/digout.reset
- J17 pad 4: /Ch4 Daughterboard/ps.ignd+ -> /Ch4 Daughterboard/digout.on1
- J17 pad 5: /Ch4 Daughterboard/ps.spare+ -> unconnected-(J17-Pad5)
- J17 pad 6: unconnected-(J17-Pad6) -> /Ch4 Daughterboard/ps.ignd+
- J17 pad 7: /Ch4 Daughterboard/digout.on1 -> /Ch4 Daughterboard/ps.spare+
- J17 pad 8: /Ch4 Daughterboard/digout.on2 -> /Ch4 Daughterboard/ps.vout+
- J17 pad 9: /Ch4 Daughterboard/digout.reset -> /Ch4 Daughterboard/reg.out+
- J8 pad 1: /Ch1 Daughterboard/reg.out+ -> /Ch1 Daughterboard/digout.rtn
- J8 pad 10: /Ch1 Daughterboard/digout.spare -> /Ch1 Daughterboard/digin.rtn
- J8 pad 11: /Ch1 Daughterboard/digout.rtn -> /Ch1 Daughterboard/digin.rtn
- J8 pad 12: /Ch1 Daughterboard/digout.rtn -> /Ch1 Daughterboard/digout.spare
- J8 pad 13: unconnected-(J8-Pad13) -> /Ch1 Daughterboard/digout.on2
- J8 pad 14: /Ch1 Daughterboard/reg.out- -> unconnected-(J8-Pad14)
- J8 pad 15: unconnected-(J8-Pad15) -> /Ch1 Daughterboard/ps.ignd-
- J8 pad 16: /Ch1 Daughterboard/ps.vout- -> /Ch1 Daughterboard/ps.spare-
- J8 pad 17: /Ch1 Daughterboard/ps.ignd- -> /Ch1 Daughterboard/ps.vout-
- J8 pad 18: /Ch1 Daughterboard/ps.spare- -> /Ch1 Daughterboard/reg.out-
- J8 pad 19: unconnected-(J8-Pad19) -> /Ch1 Daughterboard/digin.acon
- J8 pad 2: unconnected-(J8-Pad2) -> /Ch1 Daughterboard/digout.rtn
- J8 pad 20: /Ch1 Daughterboard/digin.acon -> /Ch1 Daughterboard/digin.flt1
- J8 pad 21: /Ch1 Daughterboard/digin.flt1 -> /Ch1 Daughterboard/digin.flt2
- J8 pad 22: /Ch1 Daughterboard/digin.flt2 -> /Ch1 Daughterboard/digin.spare
- J8 pad 23: /Ch1 Daughterboard/digin.spare -> unconnected-(J8-Pad23)
- J8 pad 24: /Ch1 Daughterboard/digin.rtn -> unconnected-(J8-Pad24)
- J8 pad 25: /Ch1 Daughterboard/digin.rtn -> unconnected-(J8-Pad25)
- J8 pad 26: (no net) -> unconnected-(J8-Pad26)
- J8 pad 3: /Ch1 Daughterboard/ps.vout+ -> /Ch1 Daughterboard/digout.reset
- J8 pad 4: /Ch1 Daughterboard/ps.ignd+ -> /Ch1 Daughterboard/digout.on1
- J8 pad 5: /Ch1 Daughterboard/ps.spare+ -> unconnected-(J8-Pad5)
- J8 pad 6: unconnected-(J8-Pad6) -> /Ch1 Daughterboard/ps.ignd+
- J8 pad 7: /Ch1 Daughterboard/digout.on1 -> /Ch1 Daughterboard/ps.spare+
- J8 pad 8: /Ch1 Daughterboard/digout.on2 -> /Ch1 Daughterboard/ps.vout+
- J8 pad 9: /Ch1 Daughterboard/digout.reset -> /Ch1 Daughterboard/reg.out+
Routing:
- net /Ch4 Daughterboard/ps.spare-: track 86.3 -> 70.4 mm
- net /Ch3 Daughterboard/ps.spare-: track 85.0 -> 70.4 mm
- net /Ch2 Daughterboard/ps.spare-: track 85.0 -> 70.4 mm
- net /Ch1 Daughterboard/ps.spare-: track 85.0 -> 70.4 mm
- net /Ch1 Daughterboard/ps.ignd-: track 84.5 -> 72.5 mm
- net /Ch4 Daughterboard/ps.ignd-: track 84.5 -> 72.5 mm
- net /Ch2 Daughterboard/ps.ignd-: track 84.5 -> 72.5 mm
- net /Ch3 Daughterboard/ps.ignd-: track 84.5 -> 72.5 mm
- net /Ch1 Daughterboard/ps.vout-: track 83.1 -> 71.5 mm, vias 2 -> 1
- net /Ch2 Daughterboard/ps.vout-: track 83.1 -> 71.5 mm, vias 2 -> 1
- net /Ch3 Daughterboard/ps.vout-: track 83.1 -> 71.5 mm, vias 2 -> 1
- net /Ch4 Daughterboard/ps.vout-: track 83.1 -> 71.5 mm, vias 2 -> 1
- net /Ch2 Daughterboard/digin.acon: track 87.5 -> 78.4 mm
- net /Ch3 Daughterboard/digin.acon: track 87.4 -> 78.4 mm
- net /Ch1 Daughterboard/digin.acon: track 87.4 -> 78.4 mm
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