File: daughter/rev2/ps_conn.kicad_sch (KiCad schematic)
At the start: 1 part, among them J2 61082-061400LF

Commit message: Rename versions
Parts:
- removed J2: 61082-061400LF, myparts:AMPHENOL_61082-061400LF, symbol PSC:61082-061400LF
- added J1: 61082-061400LF, myparts:AMPHENOL_61082-061400LF, symbol PSC:61082-061400LF
Connections:
- net GND: now also J1.17, J1.18, J1.19, J1.21, J1.23, J1.24, J1.25, J1.30, J1.31, J1.33, J1.36, J1.38, J1.39, J1.41, J1.44, J1.46, J1.47, J1.49, J1.52, J1.54, J1.55, J1.57, J1.59, J1.60
- new net +15V: J1.27, J1.29
- new net +5.3VA: J1.43, J1.45
- new net -15V: J1.35, J1.37
- new net -5.3VA: J1.51, J1.53
- new net dac+: J1.40
- new net dac-: J1.42
- new net dcct0+: J1.48
- new net dcct0-: J1.50
- new net dcct1+: J1.56
- new net dcct1-: J1.58
- new net digin_acon: J1.16
- new net digin_flt1: J1.14
- new net digin_flt2: J1.12
- new net digin_spare: J1.10
- new net digout_on1: J1.8
- new net digout_on2: J1.6
- new net digout_reset: J1.4
- new net digout_spare: J1.2
- new net din_iso_gnd: J1.1, J1.3, J1.5, J1.7
- new net dout_iso_gnd: J1.11, J1.13, J1.15, J1.9
- new net ps_ignd+: J1.26
- new net ps_ignd-: J1.28
- new net ps_spare+: J1.20
- new net ps_spare-: J1.22
- new net ps_vout+: J1.32
- new net ps_vout-: J1.34
