File: daughter/rev2/digin.kicad_sch (KiCad schematic)
At the start: 17 parts, among them U38 TXUN0104RUTR, U39 ADUM5240ARZ, U40 ADUM5240ARZ

Commit message: Rename versions
Parts:
- removed C104, C182, C183, C184, C185, C186: 0.1uF, Capacitor_SMD:C_0402_1005Metric, symbol Device:C_Small
- removed C187, C188: 10uF, Capacitor_SMD:C_0603_1608Metric, symbol Device:C_Small
- removed CR5, CR6: SP3006-02XTG, myparts:SOT563_LTF, symbol PSC:SP3006-02XTG
- removed R66, R67, R68, R69: 2.49K, Resistor_SMD:R_0402_1005Metric, symbol Device:R_US
- removed U38: TXUN0104RUTR, myparts:PQFP12_RUT_TEX, symbol PSC:TXUN0104RUTR
- removed U39, U40: ADUM5240ARZ, myparts:R_8_ADI-M, symbol PSC:ADUM5240ARZ
- added C102, C189, C190, C191, C192, C193: 0.1uF, Capacitor_SMD:C_0402_1005Metric, symbol Device:C_Small
- added C194, C195: 10uF, Capacitor_SMD:C_0603_1608Metric, symbol Device:C_Small
- added CR7, CR8: SP3006-02XTG, myparts:SOT563_LTF, symbol PSC:SP3006-02XTG
- added R70, R71, R72, R73: 2.49K, Resistor_SMD:R_0402_1005Metric, symbol Device:R_US
- added U41: TXUN0104RUTR, myparts:PQFP12_RUT_TEX, symbol PSC:TXUN0104RUTR
- added U42, U43: ADUM5242ARZ, myparts:R_8_ADI, symbol PSC:ADUM5242ARZ
Connections:
- net +1.8V: now also C189.1, U41.11 (VCCB)
- net +5.0V: now also C102.1, C190.1, C191.1, U41.1 (VCCA), U42.1 (VDD), U43.1 (VDD)
- net GND: now also C102.2, C189.2, C190.2, C191.2, C192.2, C193.2, C194.2, C195.2, U41.12 (~OE), U41.6 (GND), U42.4 (GND), U43.4 (GND)
- new net: C192.1, C194.1, R70.2, R72.2, U42.8 (VISO)
- new net: U41.2 (A1), U42.2 (VOA)
- new net: U41.3 (A2), U42.3 (VOB)
- new net: U41.4 (A3), U43.2 (VOA)
- new net: U41.5 (A4), U43.3 (VOB)
- new net: C193.1, C195.1, R71.2, R73.2, U43.8 (VISO)
- new net din0: U41.10 (B1Y)
- new net din0_iso: CR7.1, R70.1, U42.7 (VIA)
- new net din1: U41.9 (B2Y)
- new net din1_iso: CR7.5, R72.1, U42.6 (VIB)
- new net din2: U41.8 (B3Y)
- new net din2_iso: CR8.1, R71.1, U43.7 (VIA)
- new net din3: U41.7 (B4Y)
- new net din3_iso: CR8.5, R73.1, U43.6 (VIB)
- new net din_iso_gnd: CR7.2, CR7.4, CR8.2, CR8.4, U42.5 (GNDISO), U43.5 (GNDISO)

Commit message: Update BOM
Parts:
- C102, C189, C190, C191, C192, C193: Cost (none) -> .01
- C194, C195: Cost (none) -> .07
Changed lines of the file:
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@@
+			)
+		)
+		(property "Cost" ".01"
+			(at 173.99 39.37 0)
+			(effects
+				(font
+					(size 1.27 1.27)
+				)
+				(hide yes)
 			)
 		)
@@
 			)
 		)
+		(property "Cost" ".01"
+			(at 173.99 109.22 0)
+			(effects
+				(font
+					(size 1.27 1.27)
+				)
+				(hide yes)
+			)
+		)
 		(pin "2"
 		)
@@
 			)
 		)
+		(property "Cost" ".07"
+			(at 184.15 109.22 0)
+			(effects
+				(font
+					(size 1.27 1.27)
+				)
+				(hide yes)
+			)
+		)
 		(pin "1"
 		)
@@
 			)
 		)
+		(property "Cost" ".07"
+			(at 184.15 39.37 0)
+			(effects
+				(font
+					(size 1.27 1.27)
+				)
+				(hide yes)
+			)
+		)
 		(pin "1"
 		)
@@
 		)
 		(property "MFG_PN" "TMK105BJ104KV-F\n"
+			(at 111.76 41.91 0)
+			(effects
+				(font
+					(size 1.27 1.27)
+				)
+				(hide yes)
+			)
+		)
+		(property "Cost" ".01"
 			(at 111.76 41.91 0)
 			(effects
@@
 			)
 		)
+		(property "Cost" ".01"
+			(at 31.75 81.28 0)
+			(effects
+				(font
+					(size 1.27 1.27)
+				)
+				(hide yes)
+			)
+		)
 		(pin "2"
 		)
@@
 			)
 		)
+		(property "Cost" ".01"
+			(at 90.17 41.91 0)
+			(effects
+				(font
+					(size 1.27 1.27)
+				)
+				(hide yes)
+			)
+		)
 		(pin "2"
 		)
@@
 			(at 100.33 41.91 0)
 			(effects
+				(font
+					(size 1.27 1.27)
+				)
+				(hide yes)
+			)
+		)
+		(property "Cost" ".01"
+			(at 100.33 41.91 0)
+			(effects
