File: daughter/rev2/digout.kicad_sch (KiCad schematic)
At the start: 17 parts, among them U38 TXUN0104RUTR, U39 ADUM5240ARZ, U40 ADUM5240ARZ

Commit message: Rename versions
Parts:
- U39, U40: footprint myparts:R_8_ADI-M -> myparts:R_8_ADI
Changed lines of the file:
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@@
 			)
 		)
-		(property "Footprint" "myparts:R_8_ADI-M"
+		(property "Footprint" "myparts:R_8_ADI"
 			(at 127 50.8 0)
 			(effects
@@
 		)
 		(instances
-			(project ""
+			(project "psc_daughter_brd"
 				(path "/40891cc8-bf64-41f4-8f69-a607d7b280eb/979dab62-5512-4152-97ee-117138a961d3/84c3e299-56b9-4043-9091-ed3bb176fd4f"
 					(reference "#PWR0184")
@@
 			)
 		)
-		(property "Footprint" "myparts:R_8_ADI-M"
+		(property "Footprint" "myparts:R_8_ADI"
 			(at 127 120.65 0)
 			(effects

Commit message: Update BOM
Parts:
- C104, C182, C183, C184, C185, C186: Cost (none) -> .01
- C187, C188: Cost (none) -> .07
Changed lines of the file:
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@@
+			)
+		)
+		(property "Cost" ".01"
+			(at 111.76 41.91 0)
+			(effects
+				(font
+					(size 1.27 1.27)
+				)
+				(hide yes)
 			)
 		)
@@
 		)
 		(property "MFG_PN" "TMK105BJ104KV-F\n"
+			(at 31.75 81.28 0)
+			(effects
+				(font
+					(size 1.27 1.27)
+				)
+				(hide yes)
+			)
+		)
+		(property "Cost" ".01"
 			(at 31.75 81.28 0)
 			(effects
@@
 			)
 		)
+		(property "Cost" ".01"
+			(at 90.17 41.91 0)
+			(effects
+				(font
+					(size 1.27 1.27)
+				)
+				(hide yes)
+			)
+		)
 		(pin "2"
 		)
@@
 			)
 		)
+		(property "Cost" ".01"
+			(at 173.99 109.22 0)
+			(effects
+				(font
+					(size 1.27 1.27)
+				)
+				(hide yes)
+			)
+		)
 		(pin "2"
 		)
@@
 			)
 		)
+		(property "Cost" ".01"
+			(at 101.6 41.91 0)
+			(effects
+				(font
+					(size 1.27 1.27)
+				)
+				(hide yes)
+			)
+		)
 		(pin "2"
 		)
@@
 			)
 		)
+		(property "Cost" ".07"
+			(at 184.15 39.37 0)
+			(effects
+				(font
+					(size 1.27 1.27)
+				)
+				(hide yes)
+			)
+		)
 		(pin "1"
 		)
@@
 		)
 		(property "MFG_PN" "CL10A106MA8NRNC\n"
+			(at 184.15 109.22 0)
+			(effects
+				(font
+					(size 1.27 1.27)
+				)
+				(hide yes)
+			)
+		)
+		(property "Cost" ".07"
 			(at 184.15 109.22 0)
 			(effects
@@
 			(at 173.99 39.37 0)
 			(effects
+				(font
+					(size 1.27 1.27)
+				)
+				(hide yes)
+			)
+		)
+		(property "Cost" ".01"
+			(at 173.99 39.37 0)
+			(effects
