File: daughter/rev2/psc_daughter_brd.kicad_pcb (KiCad board)
At the start: 10 copper layers, 40 x 160 mm, 339 parts, among them J1 61082-061400LF, J2 61082-061400LF, U1 AD8221, U10 BUF634AIDR, U11 BUF634AIDR, U12 ADR1001AEZ, U13 ADS8568SPM, U14 AD8221, U15 OPA277, U16 AD8221, U17 OPA277, U18 AD8221, U19 OPA277, U2 OPA277, U20 LT3042xMSE, U21 THP210DR, U22 LT6202CS5, U23 ADA4523-1BRMZ, U24 LT6202CS5, U26 THP210DR, U27 AD8429BRZ, U3 AD8676ARZ, U31 LTC2376CDE-20, U32 LTC6655BHLS8-5, U33 AD8429BRZ, U35 LT6202CS5, U37 LTC2376CDE-20, U38 TXUN0104RUTR, U39 ADUM5240ARZ, U4 AD8676xR, U40 ADUM5240ARZ, U41 TXUN0104RUTR, U42 ADUM5242ARZ, U43 ADUM5242ARZ, U5 AD5791BRUZ, U6 AD797ARZ, U7 OPA277, U8 AD8676xR, U9 OPA277

Commit message: Add fiducials
Parts:
- added FID1: Fiducial_1mm_Mask2mm, Fiducial:Fiducial_1mm_Mask2mm, F.Cu at (141.4, 40.5)
- added FID2: Fiducial_1mm_Mask2mm, Fiducial:Fiducial_1mm_Mask2mm, F.Cu at (178.5, 33.6)
- added FID3: Fiducial_1mm_Mask2mm, Fiducial:Fiducial_1mm_Mask2mm, F.Cu at (150.5, 189.7)
- added REF**: Fiducial_1mm_Mask2mm, Fiducial:Fiducial_1mm_Mask2mm, B.Cu at (150.5, 189.7)
- added REF**: Fiducial_1mm_Mask2mm, Fiducial:Fiducial_1mm_Mask2mm, B.Cu at (178.5, 33.6)
- added REF**: Fiducial_1mm_Mask2mm, Fiducial:Fiducial_1mm_Mask2mm, B.Cu at (141.4, 40.5)
