File: daughter/rev2/psc_daughter_brd.kicad_pcb (KiCad board)
At the start: 10 copper layers, 40 x 160 mm, 345 parts, among them J1 61082-061400LF, J2 61082-061400LF, U1 AD8221, U10 BUF634AIDR, U11 BUF634AIDR, U12 ADR1001AEZ, U13 ADS8568SPM, U14 AD8221, U15 OPA277, U16 AD8221, U17 OPA277, U18 AD8221, U19 OPA277, U2 OPA277, U20 LT3042xMSE, U21 THP210DR, U22 LT6202CS5, U23 ADA4523-1BRMZ, U24 LT6202CS5, U26 THP210DR, U27 AD8429BRZ, U3 AD8676ARZ, U31 LTC2376CDE-20, U32 LTC6655BHLS8-5, U33 AD8429BRZ, U35 LT6202CS5, U37 LTC2376CDE-20, U38 TXUN0104RUTR, U39 ADUM5240ARZ, U4 AD8676xR, U40 ADUM5240ARZ, U41 TXUN0104RUTR, U42 ADUM5242ARZ, U43 ADUM5242ARZ, U5 AD5791BRUZ, U6 AD797ARZ, U7 OPA277, U8 AD8676xR, U9 OPA277

Commit message: Add gerbers
Parts:
- removed FID1, FID2, FID3, REF** (x3): Fiducial_1mm_Mask2mm, Fiducial:Fiducial_1mm_Mask2mm
- added D10: LED, LED_SMD:LED_0603_1608Metric, F.Cu at (164.9, 189.1)
- added D11: LED, LED_SMD:LED_0603_1608Metric, F.Cu at (166.8, 189.1)
- added R57: 220, Resistor_SMD:R_0603_1608Metric, F.Cu at (164.9, 185.8)
- added R84: 220, Resistor_SMD:R_0603_1608Metric, F.Cu at (166.8, 185.8)
- moved TP4 5.45 mm to (155.7, 187.1)
Connections:
- J2 pad 57: GND -> Net-(J2-Pad57)
- J2 pad 59: GND -> Net-(J2-Pad59)
Routing:
- net Net-(J2-Pad57): track 0.00 -> 17.5 mm, vias 0 -> 1
- net Net-(J2-Pad59): track 0.00 -> 16.1 mm, vias 0 -> 1
- net Net-(D11-A): track 0.00 -> 1.69 mm
- net Net-(D10-A): track 0.00 -> 1.69 mm
- net GND: track 451.7 -> 450.3 mm
- net /FPGA connector/mon_busy: track 32.2 -> 31.0 mm, vias 1 -> 3
Other:
- board text added: "1. BOARD SIZE: 160.0 mm x 40.0 mm. 2. LAYER COUNT: 10 LAYERS. 3. MATERIAL: FR-4, SHENGYI S1000-2M OR APPROVED EQUIVALENT, Tg = 170°C. 4. FINISHED BOARD THICKNESS: 1.60 mm. 5. COPPER WEIGHT: OUTER LAYERS: 1 oz Cu. INNER LAYERS: 1 oz Cu. 6. MINIMUM TRACE / SPACE: 5 mil / 5 mil. 7. MINIMUM HOLE SIZE: 0.30 mm. 8. PLATED HOLE COPPER: 20 µm MINIMUM / STANDARD FABRICATION PROCESS. 9. SOLDER MASK: GREEN,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"
- board text added: "Fabrication Notes"
