File: daughter/rev2/fpga_conn.kicad_sch (KiCad schematic)
At the start: 1 part, among them J2 61082-061400LF

Commit message: Add gerbers
Parts:
- added D10, D11: LED, LED_SMD:LED_0603_1608Metric, symbol Device:LED
- added R57, R84: 220, Resistor_SMD:R_0603_1608Metric, symbol Device:R_US
Connections:
- net GND: now also D10.1 (K), D11.1 (K); no longer J2.57, J2.59
- new net: D11.2 (A), R84.2
- new net: J2.57, R57.1
- new net: D10.2 (A), R57.2
- new net: J2.59, R84.1
